File: FS-SensorBoard.kicad_pcb (KiCad board)
At the start: 2 copper layers, 97 x 70 mm, 58 parts, among them J1 USB_B, M3_1 MountingHole, M3_2 MountingHole, M3_3 MountingHole, M3_4 MountingHole, U1 CH340C, U2 ESP32-WROOM-32, U3 TJA1051TK-3, U4 LM2576S-3.3, U5 LM2576S-5

Commit message: Edited footprint
Parts:
- removed Damper_1, Damper_2, Damper_3, Damper_4: Conn_01x02, Connector_JST:JST_XH_B2B-XH-A_1x02_P2.50mm_Vertical
- removed R17, R18, R19, R20: 1000k, Resistor_SMD:R_1206_3216Metric_Pad1.30x1.75mm_HandSolder
- added D3: LED, LED_SMD:LED_1206_3216Metric_Pad1.42x1.75mm_HandSolder, F.Cu at (228.4, 82.8)
- added D4: LED, LED_SMD:LED_1206_3216Metric_Pad1.42x1.75mm_HandSolder, F.Cu at (228.4, 86.2)
- added Damper1: Conn_01x03, Connector_JST:JST_XH_B3B-XH-A_1x03_P2.50mm_Vertical, F.Cu at (213.6, 61.1)
- added Damper2: Conn_01x03, Connector_JST:JST_XH_B3B-XH-A_1x03_P2.50mm_Vertical, F.Cu at (213.6, 68.9)
- added Damper3: Conn_01x03, Connector_JST:JST_XH_B3B-XH-A_1x03_P2.50mm_Vertical, F.Cu at (213.6, 76.7)
- added Damper4: Conn_01x03, Connector_JST:JST_XH_B3B-XH-A_1x03_P2.50mm_Vertical, F.Cu at (225.6, 45.5)
- added Q1: SS8050, Package_TO_SOT_SMD:SOT-23, F.Cu at (254.3, 61.3)
- added Q2: SS8050, Package_TO_SOT_SMD:SOT-23, F.Cu at (254.3, 65.9)
- added R22: 47R, Resistor_SMD:R_1206_3216Metric_Pad1.30x1.75mm_HandSolder, F.Cu at (248.9, 43.8)
- added R23: 1k, Resistor_SMD:R_1206_3216Metric_Pad1.30x1.75mm_HandSolder, F.Cu at (248.9, 47.1)
- added R24: 4k7, Resistor_SMD:R_1206_3216Metric_Pad1.30x1.75mm_HandSolder, F.Cu at (248.9, 50.4)
- added R25: 1k, Resistor_SMD:R_1206_3216Metric_Pad1.30x1.75mm_HandSolder, F.Cu at (248.9, 53.7)
- added R26: 4k7, Resistor_SMD:R_1206_3216Metric_Pad1.30x1.75mm_HandSolder, F.Cu at (248.9, 56.9)
- added R27: 1k, Resistor_SMD:R_1206_3216Metric_Pad1.30x1.75mm_HandSolder, F.Cu at (248.9, 60.2)
- added R28: 4k7, Resistor_SMD:R_1206_3216Metric_Pad1.30x1.75mm_HandSolder, F.Cu at (248.9, 63.5)
- added U6: TXS0108EPW, Package_SO:TSSOP-20_4.4x6.5mm_P0.65mm, F.Cu at (214.9, 85.2)
- Accelerometer1: value Conn_01x02 -> Conn_01x04; footprint Connector_JST:JST_XH_B2B-XH-A_1x02_P2.50mm_Vertical -> Connector_JST:JST_XH_B4B-XH-A_1x04_P2.50mm_Vertical
- Brake_Press1, Brake_Temp1, Flow_Sensor1, LV_Temp1, LV_Volt1, Water_Temp1: value Conn_01x02 -> Conn_01x03; footprint Connector_JST:JST_XH_B2B-XH-A_1x02_P2.50mm_Vertical -> Connector_JST:JST_XH_B3B-XH-A_1x03_P2.50mm_Vertical
- C10, C9: value 1000u -> 330u
- CAN_1: value Conn_01x02_Pin -> Conn_01x04; footprint Connector_JST:JST_XH_B2B-XH-A_1x02_P2.50mm_Vertical -> Connector_JST:JST_XH_B4B-XH-A_1x04_P2.50mm_Vertical
- R1: value 100k -> 1k
- R10: value 1000k -> 1k
- R11, R12, R9: value 1000k -> 4k7
- R13, R14: value 220k -> 4k7
- R15, R16: value 220k -> 10k
- R2: value 470k -> 10k
- R4, R5, R6, R7: value 220k -> 1k
- R8: value 470k -> 47R
- U2: footprint RF_Module:ESP32-WROOM-32 -> Library:ESP32-WROOM-32-LongPad
- moved R9 152.2 mm to (243.0, 43.8), turned to 0 degrees
- moved R15 149.5 mm to (243.0, 63.5), turned to 0 degrees
- moved M3_4 145.0 mm to (238.0, 80.4)
- moved R8 143.9 mm to (237.0, 66.8), turned to 0 degrees
- moved R2 142.5 mm to (237.0, 47.1)
- moved R4 142.2 mm to (237.0, 53.7), turned to 0 degrees
- moved R10 141.5 mm to (243.0, 47.1), turned to 0 degrees
- moved R1 141.0 mm to (237.0, 43.8), turned to 0 degrees
- moved R14 140.4 mm to (243.0, 60.2), turned to 0 degrees
- moved C8 138.3 mm to (254.9, 50.5), turned to 0 degrees
- moved LV_Volt1 133.5 mm to (225.6, 68.9)
- moved R3 133.5 mm to (237.0, 50.4), turned to 0 degrees
- moved R5 131.6 mm to (237.0, 56.9), turned to 0 degrees
- moved R13 131.5 mm to (243.0, 56.9), turned to 0 degrees
- moved U3 130.9 mm to (245.1, 86.4), turned to 0 degrees
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Connections:
- net /CAN_RX renamed CAN_RX
- net /CAN_TX renamed CAN_TX
- net /E-RX renamed E-RX
- net /E-TX renamed E-TX
- Accelerometer1 pad 1: /I2C_1 -> GND
- Accelerometer1 pad 2: /I2C_2 -> +5V
- Brake_Press1 pad 1: Net-(Brake_Press1-Pin_1) -> +5V
- Brake_Temp1 pad 1: Net-(Brake_Temp1-Pin_1) -> +5V
- CAN_1 pad 1: Net-(CAN_1-Pin_1) -> +5V
- Flow_Sensor1 pad 1: Net-(Flow_Sensor1-Pin_1) -> +5V
- LV_Temp1 pad 1: /ADC1_3 -> +5V
- LV_Volt1 pad 1: Net-(LV_Volt1-Pin_1) -> +12V
- R1 pad 1: /ADC1_0 -> GND
- R1 pad 2: GND -> ADC1_0
- R10 pad 1: Net-(Brake_Press1-Pin_1) -> GND
- R10 pad 2: /ADC1_5 -> ADC2_7
- R11 pad 1: Net-(Water_Temp1-Pin_1) -> ADC2_4
- R11 pad 2: /ADC1_6 -> Net-(Damper1-Pin_3)
- R12 pad 1: Net-(Flow_Sensor1-Pin_1) -> ADC2_5
- R12 pad 2: /ADC1_7 -> Net-(Damper2-Pin_3)
- R13 pad 1: /ADC2_4 -> ADC2_6
- R13 pad 2: GND -> Net-(Damper3-Pin_3)
- R14 pad 1: /ADC2_5 -> ADC2_7
- R14 pad 2: GND -> Net-(Damper4-Pin_3)
- R15 pad 1: /ADC2_6 -> RTS
- R15 pad 2: GND -> Net-(Q2-B)
- R16 pad 1: /ADC2_7 -> DTR
- R16 pad 2: GND -> Net-(Q1-B)
- R2 pad 1: Net-(R2-Pad1) -> ADC1_0
- R2 pad 2: /ADC1_0 -> Net-(LV_Volt1-Pin_3)
- R3 pad 1: GND -> ADC1_3
- R3 pad 2: /ADC1_3 -> GND
- R4 pad 1: /ADC1_4 -> GND
- R4 pad 2: GND -> ADC1_5
- R5 pad 1: /ADC1_5 -> GND
- R5 pad 2: GND -> ADC2_4
- R6 pad 1: /ADC1_6 -> GND
- R6 pad 2: GND -> ADC2_5
- R7 pad 1: /ADC1_7 -> GND
- R7 pad 2: GND -> ADC2_6
- R8 pad 1: Net-(LV_Volt1-Pin_1) -> +3V3
- R8 pad 2: Net-(R2-Pad1) -> Net-(D3-A)
- R9 pad 1: Net-(Brake_Temp1-Pin_1) -> ADC1_5
- R9 pad 2: /ADC1_4 -> Net-(Brake_Press1-Pin_3)
- U1 pad 13: unconnected-(U1-~{DTR}-Pad13) -> DTR
- U1 pad 14: unconnected-(U1-~{RTS}-Pad14) -> RTS
- U2 pad 12: /ADC2_7 -> ADC2_7
- U2 pad 13: /ADC2_6 -> ADC2_6
- U2 pad 14: /ADC2_5 -> ADC2_5
- U2 pad 16: /ADC2_4 -> ADC2_4
- U2 pad 25: unconnected-(U2-IO0-Pad25) -> IO_0
- U2 pad 36: /I2C_1 -> I2C_1
- U2 pad 37: /I2C_2 -> I2C_2
- U2 pad 4: /ADC1_0 -> ADC1_0
- U2 pad 5: /ADC1_3 -> ADC1_3
- U2 pad 6: /ADC1_6 -> ADC1_6
- U2 pad 7: /ADC1_7 -> ADC1_7
- U2 pad 8: /ADC1_4 -> ADC1_4
- U2 pad 9: /ADC1_5 -> ADC1_5
- U3 pad 6: Net-(CAN_1-Pin_1) -> Net-(CAN_1-Pin_3)
- Water_Temp1 pad 1: Net-(Water_Temp1-Pin_1) -> +5V
Routing:
- net +5V: track 128.7 -> 2.67 mm, vias 5 -> 0
- net +3V3: track 125.8 -> 15.3 mm, vias 3 -> 0
- net /I2C_1: track 75.4 -> 0.00 mm, vias 1 -> 0
- net /ADC2_6: track 74.6 -> 0.00 mm
- net /I2C_2: track 70.7 -> 0.00 mm, vias 1 -> 0
- net /ADC1_0: track 69.4 -> 0.00 mm
- net /ADC1_4: track 66.3 -> 0.00 mm
- net /ADC2_5: track 63.9 -> 0.00 mm
- net /ADC2_4: track 57.8 -> 0.00 mm
- net /ADC1_3: track 56.1 -> 0.00 mm
- net /ADC1_5: track 55.3 -> 0.00 mm
- net CAN_TX: track 48.0 -> 0.00 mm
- net CAN_RX: track 46.2 -> 0.00 mm
- net /ADC1_6: track 36.1 -> 0.00 mm
- net +12V: track 36.1 -> 0.00 mm, vias 2 -> 0
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Other:
- board outline removed
- board text removed: "CANH CANL"
- board text removed: "D- D+"
- board text removed: "E-TX E-RX"
- board text removed: "I2C _2 I2C _1 TX RX"
- board text removed: "I2C_2 I2C_1"
- board text removed: "Input GND"

Commit message: V2.Garbage.0
Parts:
- removed LV_Volt1: Conn_01x03, Connector_JST:JST_XH_B3B-XH-A_1x03_P2.50mm_Vertical
- added R17: 1k, Resistor_SMD:R_1206_3216Metric_Pad1.30x1.75mm_HandSolder, F.Cu at (109.6, 43.3)
- C10, C9: footprint Capacitor_SMD:C_1206_3216Metric_Pad1.33x1.80mm_HandSolder -> Capacitor_SMD:C_1808_4520Metric_Pad1.72x2.30mm_HandSolder
- L1, L2: footprint Inductor_SMD:L_1206_3216Metric_Pad1.22x1.90mm_HandSolder -> Inductor_SMD:L_Bourns-SRN4018
- R22: value 47R -> 4k
- R8: value 47R -> 2k
- moved C8 155.0 mm to (100.1, 57.1), turned to -90 degrees
- moved C10 154.9 mm to (102.0, 81.9), turned to 180 degrees
- moved CAN_1 153.6 mm to (93.6, 56.3), turned to 90 degrees
- moved R23 150.9 mm to (99.8, 70.0), turned to 90 degrees
- moved R24 149.8 mm to (99.8, 64.6), turned to 90 degrees
- moved Accelerometer1 149.3 mm to (100.6, 35.9)
- moved C7 146.6 mm to (113.4, 85.7), turned to 90 degrees
- moved U3 146.6 mm to (102.5, 52.5), turned to 180 degrees
- moved R22 145.8 mm to (105.9, 72.2)
- moved M3_4 145.1 mm to (94.0, 98.0)
- moved R25 143.5 mm to (105.5, 57.4)
- moved R27 143.4 mm to (105.5, 61.1)
- moved R26 139.3 mm to (109.6, 55.0), turned to 90 degrees
- moved R28 139.3 mm to (109.6, 63.5), turned to -90 degrees
- moved C9 132.5 mm to (125.4, 82.1), turned to 180 degrees
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Connections:
- Brake_Temp1 pad 3: ADC1_3 -> Net-(Brake_Temp1-Pin_3)
- C3 pad 2: Net-(U2-EN) -> EN
- Q2 pad 3: IO0 -> IO_0
- R2 pad 2: Net-(LV_Volt1-Pin_3) -> +12V
- R21 pad 2: Net-(U2-EN) -> EN
- U2 pad 3: Net-(U2-EN) -> EN
Routing:
- net +5V: track 2.67 -> 294.5 mm, vias 0 -> 9
- net +3V3: track 15.3 -> 127.6 mm, vias 0 -> 4
- net +12V: track 0.00 -> 102.5 mm, vias 0 -> 3
- net ADC2_7: track 0.00 -> 76.6 mm
- net ADC2_6: track 0.00 -> 75.4 mm
- net I2C_2: track 0.00 -> 60.7 mm, vias 0 -> 2
- net I2C_1: track 0.00 -> 59.1 mm, vias 0 -> 2
- net ADC1_4: track 0.00 -> 50.8 mm, vias 0 -> 2
- net ADC2_5: track 0.00 -> 50.7 mm, vias 0 -> 2
- net EN: track 0.00 -> 42.7 mm, vias 0 -> 2
- net ADC1_7: track 0.00 -> 37.9 mm, vias 0 -> 2
- net CAN_TX: track 0.00 -> 36.2 mm
- net ADC1_6: track 0.00 -> 36.2 mm, vias 0 -> 2
- net CAN_RX: track 0.00 -> 35.2 mm
- net ADC2_4: track 0.00 -> 32.4 mm, vias 0 -> 2
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Other:
- board outline added: 97 x 70 mm
- board text added: "3.3V"
- board text added: "5V"
- board text added: "LVV LVT Water_T Flow BkT BkP CAN_RX CAN_TX Damper4 Damper3 Damper2"
- board text removed: "LVV LVT Water_T Flow BrakeT BrakeP CAN_RX CAN_TX Damper4 Damper3 Damper2"
