File: FS-SensorBoard.kicad_sch (KiCad schematic)
At the start: 62 parts, among them J1 USB_B, M3_1 MountingHole, M3_2 MountingHole, M3_3 MountingHole, M3_4 MountingHole, U1 CH340C, U2 ESP32-WROOM-32, U3 TJA1051TK-3, U4 LM2576S-3.3, U5 LM2576S-5, U6 TXS0108EPW

Commit message: Completed Schematics
Parts:
- removed Accelerometer1, Brake_Press1, Damper_1, Damper_2, Damper_3, Damper_4, Flow_Sensor1, LV_Temp1, Water_Temp1: Conn_01x02, Connector_JST:JST_XH_B2B-XH-A_1x02_P2.50mm_Vertical, symbol Connector_Generic:Conn_01x02
- removed CAN_1: Conn_01x02_Pin, Connector_JST:JST_XH_B2B-XH-A_1x02_P2.50mm_Vertical, symbol Connector:Conn_01x02_Pin
- removed R17, R18, R19, R20: 1000k, Resistor_SMD:R_1206_3216Metric_Pad1.30x1.75mm_HandSolder, symbol Device:R
- added Accelerometer1: Conn_01x04, Connector_JST:JST_XH_B3B-XH-A_1x03_P2.50mm_Vertical, symbol Connector_Generic:Conn_01x04
- added Brake_Press1, Damper1, Damper2, Damper3, Damper4, Flow_Sensor1, LV_Temp1, Water_Temp1: Conn_01x03, symbol Connector_Generic:Conn_01x03
- added CAN_1: Conn_01x04, symbol Connector_Generic:Conn_01x04
- added Q1, Q2: SS8050, Package_TO_SOT_SMD:SOT-23, symbol Transistor_BJT:SS8050
- added R23, R25, R27: 1k, Resistor_SMD:R_1206_3216Metric_Pad1.30x1.75mm_HandSolder, symbol Device:R
- added R24, R26, R28: 4k7, Resistor_SMD:R_1206_3216Metric_Pad1.30x1.75mm_HandSolder, symbol Device:R
- R1: value 100k -> 1k
- R10: value 1000k -> 1k
- R11, R12, R9: value 1000k -> 4k7
- R13, R14: value 220k -> 4k7
- R15, R16: value 220k -> 10k; footprint Resistor_SMD:R_1206_3216Metric_Pad1.30x1.75mm_HandSolder -> (none)
- R2: value 470k -> 10k
- R4, R5, R6, R7: value 220k -> 1k
Connections:
- net +3V3: now also U6.2 (VCCA)
- net +5V: now also Brake_Temp1.1 (Pin_1), U6.19 (VCCB), Accelerometer1.2 (Pin_2), Brake_Press1.1 (Pin_1), CAN_1.1 (Pin_1), Damper1.1 (Pin_1), Damper2.1 (Pin_1), Damper3.1 (Pin_1), Damper4.1 (Pin_1), Flow_Sensor1.1 (Pin_1), LV_Temp1.1 (Pin_1), Water_Temp1.1 (Pin_1)
- net ADC1_4: now also R23.2, R24.1; no longer R4.1, R9.2
- net ADC1_5: now also R4.2, R9.1; no longer R10.2, R5.1
- net ADC1_6: now also R25.2, R26.1; no longer R11.2, R6.1
- net ADC1_7: now also R27.2, R28.1; no longer R12.2, R7.1
- net ADC2_4: now also R11.1, R5.2; no longer R13.1
- net ADC2_5: now also R12.1, R6.2; no longer R14.1
- net ADC2_6: now also R13.1, R7.2; no longer R15.1
- net ADC2_7: now also R10.2, R14.1; no longer R16.1
- net GND: now also R10.1, R4.1, R5.1, R6.1, R7.1, U6.10 (OE), U6.11 (GND), Accelerometer1.1 (Pin_1), Brake_Press1.2 (Pin_2), CAN_1.4 (Pin_4), Damper1.2 (Pin_2), Damper2.2 (Pin_2), Damper3.2 (Pin_2), Damper4.2 (Pin_2), Flow_Sensor1.2 (Pin_2), LV_Temp1.2 (Pin_2), R23.1, R25.1, R27.1, Water_Temp1.2 (Pin_2); no longer R13.2, R14.2, R15.2, R16.2, R4.2, R5.2, R6.2, R7.2
- net I2C_1: now also U6.1 (A1)
- net I2C_2: now also U6.3 (A2)
- net IO_0: now reaches U2.25 (IO0)
- net DTR: now reaches U1.13 (~{DTR})
- net DTR: now also R16.1, Q2.2 (E)
- net RTS: now reaches U1.14 (~{RTS})
- net RTS: now also R15.1, Q1.2 (E)
- net at U3.6 (CANL): now also CAN_1.3 (Pin_3)
- net at U3.7 (CANH): now also CAN_1.2 (Pin_2)
- net I2C_SDA: now reaches U6.18 (B2)
- net I2C_SDA: now also Accelerometer1.4 (Pin_4)
- net I2C_SCL: now reaches U6.20 (B1)
- net I2C_SCL: now also Accelerometer1.3 (Pin_3)
- new net: Damper4.3 (Pin_3), R14.2
- new net: Brake_Press1.3 (Pin_3), R9.2
- new net: LV_Temp1.3 (Pin_3), R24.2
- new net: R26.2, Water_Temp1.3 (Pin_3)
- new net: Q1.1 (B), R16.2
- new net: Q2.1 (B), R15.2
- new net: Damper3.3 (Pin_3), R13.2
- new net: Damper1.3 (Pin_3), R11.2
- new net: Damper2.3 (Pin_3), R12.2
- new net: Flow_Sensor1.3 (Pin_3), R28.2
- new net EN: Q1.3 (C)
- new net IO0: Q2.3 (C)
- no-connect marks 23 -> 32
Other:
- note removed: "3-SCL"
- note removed: "4-SDA"
- moved on the sheet: C3, C4, C5, C8, R21, U2, U3, U6

Commit message: Edited footprint
Parts:
- Accelerometer1: footprint Connector_JST:JST_XH_B3B-XH-A_1x03_P2.50mm_Vertical -> Connector_JST:JST_XH_B4B-XH-A_1x04_P2.50mm_Vertical
- Brake_Press1, Brake_Temp1, Damper1, Damper2, Damper3, Damper4, Flow_Sensor1, LV_Temp1, LV_Volt1, Water_Temp1: footprint (none) -> Connector_JST:JST_XH_B3B-XH-A_1x03_P2.50mm_Vertical
- CAN_1: footprint (none) -> Connector_JST:JST_XH_B4B-XH-A_1x04_P2.50mm_Vertical
- D3, D4: footprint (none) -> LED_SMD:LED_1206_3216Metric_Pad1.42x1.75mm_HandSolder
- R15, R16: footprint (none) -> Resistor_SMD:R_1206_3216Metric_Pad1.30x1.75mm_HandSolder
- U2: footprint RF_Module:ESP32-WROOM-32 -> Library:ESP32-WROOM-32-LongPad
Changed lines of the file:
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@@
 			)
 		)
-		(property "Footprint" "RF_Module:ESP32-WROOM-32"
+		(property "Footprint" "Library:ESP32-WROOM-32-LongPad"
 			(at 139.7 175.26 0)
 			(effects
@@
 			)
 		)
-		(property "Footprint" ""
+		(property "Footprint" "Connector_JST:JST_XH_B3B-XH-A_1x03_P2.50mm_Vertical"
 			(at 43.18 127 0)
 			(effects
@@
 			)
 		)
-		(property "Footprint" "Connector_JST:JST_XH_B3B-XH-A_1x03_P2.50mm_Vertical"
+		(property "Footprint" "Connector_JST:JST_XH_B4B-XH-A_1x04_P2.50mm_Vertical"
 			(at 85.09 87.63 0)
 			(effects
@@
 			)
 		)
-		(property "Footprint" ""
+		(property "Footprint" "Connector_JST:JST_XH_B3B-XH-A_1x03_P2.50mm_Vertical"
 			(at 85.09 167.64 0)
 			(effects
@@
 			)
 		)
-		(property "Footprint" ""
+		(property "Footprint" "Connector_JST:JST_XH_B3B-XH-A_1x03_P2.50mm_Vertical"
 			(at 43.18 67.31 0)
 			(effects
@@
 			)
 		)
-		(property "Footprint" ""
+		(property "Footprint" "Connector_JST:JST_XH_B3B-XH-A_1x03_P2.50mm_Vertical"
 			(at 43.18 106.68 0)
 			(effects
@@
 			)
 		)
-		(property "Footprint" ""
+		(property "Footprint" "Resistor_SMD:R_1206_3216Metric_Pad1.30x1.75mm_HandSolder"
 			(at 176.53 37.338 90)
 			(effects
@@
 			)
 		)
-		(property "Footprint" ""
+		(property "Footprint" "LED_SMD:LED_1206_3216Metric_Pad1.42x1.75mm_HandSolder"
 			(at 245.11 60.96 0)
 			(effects
@@
 			)
 		)
-		(property "Footprint" ""
+		(property "Footprint" "Connector_JST:JST_XH_B3B-XH-A_1x03_P2.50mm_Vertical"
 			(at 85.09 147.32 0)
 			(effects
@@
 			)
 		)
-		(property "Footprint" ""
+		(property "Footprint" "Resistor_SMD:R_1206_3216Metric_Pad1.30x1.75mm_HandSolder"
 			(at 176.53 48.768 90)
 			(effects
@@
 			)
 		)
-		(property "Footprint" ""
+		(property "Footprint" "Connector_JST:JST_XH_B3B-XH-A_1x03_P2.50mm_Vertical"
 			(at 85.09 127 0)
 			(effects
@@
 			)
 		)
-		(property "Footprint" ""
+		(property "Footprint" "Connector_JST:JST_XH_B3B-XH-A_1x03_P2.50mm_Vertical"
 			(at 43.18 167.64 0)
 			(effects
@@
 			)
 		)
-		(property "Footprint" ""
+		(property "Footprint" "Connector_JST:JST_XH_B4B-XH-A_1x04_P2.50mm_Vertical"
 			(at 276.86 129.54 0)
 			(effects
@@
 			)
 		)
-		(property "Footprint" ""
+		(property "Footprint" "LED_SMD:LED_1206_3216Metric_Pad1.42x1.75mm_HandSolder"
 			(at 245.11 53.34 0)
 			(effects
@@
 			)
 		)
-		(property "Footprint" ""
+		(property "Footprint" "Connector_JST:JST_XH_B3B-XH-A_1x03_P2.50mm_Vertical"
 			(at 85.09 106.68 0)
 			(effects
@@
 			)
 		)
-		(property "Footprint" ""
+		(property "Footprint" "Connector_JST:JST_XH_B3B-XH-A_1x03_P2.50mm_Vertical"
 			(at 43.18 147.32 0)
 			(effects
@@
 			)
 		)
-		(property "Footprint" ""
+		(property "Footprint" "Connector_JST:JST_XH_B3B-XH-A_1x03_P2.50mm_Vertical"
 			(at 43.18 87.63 0)
 			(effects

Commit message: V2.Garbage.0
Parts:
- removed LV_Volt1: Conn_01x03, Connector_JST:JST_XH_B3B-XH-A_1x03_P2.50mm_Vertical, symbol Connector_Generic:Conn_01x03
- added R17: 1k, Resistor_SMD:R_1206_3216Metric_Pad1.30x1.75mm_HandSolder, symbol Device:R
- C10, C9: footprint Capacitor_SMD:C_1206_3216Metric_Pad1.33x1.80mm_HandSolder -> Capacitor_SMD:C_1808_4520Metric_Pad1.72x2.30mm_HandSolder
- L1, L2: footprint Inductor_SMD:L_1206_3216Metric_Pad1.22x1.90mm_HandSolder -> Inductor_SMD:L_Bourns-SRN4018
- R22: value 47R -> 4k
- R8: value 47R -> 2k
Connections:
- net IO0 is gone; now on net IO_0: Q2.3 (C)
- net +12V: now also R2.2
- net ADC1_3: now also R17.1; no longer Brake_Temp1.3 (Pin_3)
- net EN: now also C3.2, R21.2, U2.3 (EN)
- new net: Brake_Temp1.3 (Pin_3), R17.2
Other:
- moved on the sheet: R1, R2, R21
